File: misc/power_shield/power_shield_eagle_source/power_shield.brd (EAGLE design)
At the start: 68.6 x 55.9 mm, 29 parts

Commit message: Seperated the electronics
Parts:
- L1, L2: value 100mH -> 0.1mH
Changed lines of the file:
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@@
 <element name="C3" library="rcl" package="150CLZ-1010" value="100uF" x="62.23" y="22.86" rot="R90"/>
 <element name="C4" library="rcl" package="150CLZ-1010" value="100uF" x="62.23" y="36.83" rot="R90"/>
-<element name="L1" library="rcl" package="6000-XXXX-RC" value="100mH" x="45.72" y="24.13" rot="R180"/>
-<element name="L2" library="rcl" package="6000-XXXX-RC" value="100mH" x="45.72" y="38.1" rot="R180"/>
+<element name="L1" library="rcl" package="6000-XXXX-RC" value="0.1mH" x="45.72" y="24.13" rot="R180"/>
+<element name="L2" library="rcl" package="6000-XXXX-RC" value="0.1mH" x="45.72" y="38.1" rot="R180"/>
 <element name="U$1" library="mylib" package="UNO32_SHIELD" value="UNO32_SHIELD" x="64.77" y="3.81"/>
 <element name="U$2" library="mylib" package="TO-220-5" value="LM2576-5.0" x="53.34" y="36.83"/>
